Commit message: realsense_gazebo

File: rover_description/urdf/husky.urdf.xacro (robot description, xacro)
@@ -175,5 +175,5 @@
   </joint>
   <!-- Spawn user right realsense -->
-  <link name="Central_D435_link">
+  <!--link name="Central_D435_link">
     <visual>
       <geometry>
@@ -181,11 +181,14 @@
       </geometry>
     </visual>
-  </link>
+  </link-->
   <!-- Attach user fight realsense to base link -->
+  <link name="Central_D435_link"/>
   <joint name="Central_D435" type="fixed">
-    <origin xyz="0.254623 -0.01 0.3720229" rpy="1.5707963268 0.0 1.5707963268" />
+    <!--origin xyz="0.254623 -0.01 0.3720229" rpy="1.5707963268 0.0 1.5707963268" /-->
+    <origin xyz="0.254623 -0.01 0.3720229" rpy="0.0 0.0 0.0" />
     <parent link="base_link" />
     <child link="Central_D435_link" />
   </joint>
+    <xacro:intel_realsense_mount prefix="camera" topic="realsense" parent_link="Central_D435_link"/>
   <!-- Spawn user right realsense -->
   <link name="T265_link">

Commit message: move_sequences

File: rover_description/urdf/husky.urdf.xacro (robot description, xacro)
@@ -190,4 +190,7 @@
     <child link="T265_link" />
   </joint>
+  <!--xacro:realsense_T265 sensor_name="camera" parent_link="T265_link" rate="30.0">
+    <origin rpy="0 0 0" xyz="0 0 0.5"/>
+  </xacro:realsense_T265-->
   <!-- Spawn user bracket_t265nd435_2 -->
   <link name="Bracket_t265nd435_link">
